File: hardware/LEC/ADC_Power_Circuit.kicad_sch (KiCad schematic)
At the start: 8 parts, among them U7 L78L33ACZ, U8 L78L33ACZ

Commit message: Updated schematic documentation, more production files
Parts:
- C1: DigiKey (none) -> https://www.digikey.com/en/products/detail/murata-electroni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; Digikey https://www.digikey.com/en/products/detail/murata-electroni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 -> (none)
- U7, U8: DigiKey (none) -> https://www.digikey.com/en/products/detail/stmicroelectroni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
Changed lines of the file:
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@@
       (effects (font (size 1.27 1.27)) hide)
     )
-    (property "Digikey" "https://www.digikey.com/en/products/detail/murata-electronics/GRM3195C1H104JA05D/13531811" (at 87.63 95.25 0)
+    (property "DigiKey" "https://www.digikey.com/en/products/detail/murata-electronics/GRM3195C1H104JA05D/13531811" (at 87.63 95.25 0)
       (effects (font (size 1.27 1.27)) hide)
     )
@@
       (effects (font (size 1.27 1.27) italic) hide)
     )
+    (property "DigiKey" "https://www.digikey.com/en/products/detail/stmicroelectronics/L78L33ACZ/1038304" (at 215.9 71.12 0)
+      (effects (font (size 1.27 1.27)) hide)
+    )
     (pin "1")
     (pin "2")
@@
       (effects (font (size 1.27 1.27)) hide)
     )
-    (property "Digikey" "https://www.digikey.com/en/products/detail/murata-electronics/GRM3195C1H104JA05D/13531811" (at 209.55 96.52 0)
+    (property "DigiKey" "https://www.digikey.com/en/products/detail/murata-electronics/GRM3195C1H104JA05D/13531811" (at 209.55 96.52 0)
       (effects (font (size 1.27 1.27)) hide)
     )
@@
       (effects (font (size 1.27 1.27)) hide)
     )
-    (property "Digikey" "https://www.digikey.com/en/products/detail/murata-electronics/GRM3195C1H104JA05D/13531811" (at 209.55 109.22 0)
+    (property "DigiKey" "https://www.digikey.com/en/products/detail/murata-electronics/GRM3195C1H104JA05D/13531811" (at 209.55 109.22 0)
       (effects (font (size 1.27 1.27)) hide)
     )
@@
       (effects (font (size 1.27 1.27) italic) hide)
     )
+    (property "DigiKey" "https://www.digikey.com/en/products/detail/stmicroelectronics/L78L33ACZ/1038304" (at 82.55 71.12 0)
+      (effects (font (size 1.27 1.27)) hide)
+    )
     (pin "1")
     (pin "2")
@@
       (effects (font (size 1.27 1.27)) hide)
     )
-    (property "Digikey" "https://www.digikey.com/en/products/detail/murata-electronics/GRM3195C1H104JA05D/13531811" (at 87.63 107.95 0)
-      (effects (font (size 1.27 1.27)) hide)
-    )
+    (property "DigiKey" "https://www.digikey.com/en/products/detail/murata-electronics/GRM3195C1H104JA05D/13531811" (at 87.63 107.95 0)
+      (effects (font (size 1.27 1.27)) hide)
+    )
