File: hardware/LEC/LEC.kicad_pcb (KiCad board)
At the start: 4 copper layers, 152.9 x 77.2 mm, 71 parts, among them J1 54-00278, J10 Conn_01x02, J11 54-00278, J12 54-00278, J13 54-00278, J14 54-00278, J2 54-00278, J3 54-00278, J4 54-00278, J5 54-00278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

Commit message: Updated schematic documentation, more production files
Parts:
- C23, C26: value C -> 10n
