File: hardware/XBeeBreakoutBoard/XBeeBreakoutBoard.kicad_pcb (KiCad board)
At the start: 2 copper layers, 47.5 x 62.9 mm, 13 parts, among them J1 Conn_01x02, J2 Conn_01x10_Socket, J4 Conn_01x10_Socket, J5 Conn_01x05_Pin, U1 XB3-24Z8PT-J

Commit message: XBee Breakout production files
Parts:
- moved REF** 0.40 mm to (156.8, 100.0)
Connections:
- J2 pad 9: Net-(J2-Pin_9) -> GND
- U1 pad 10: Net-(J2-Pin_9) -> GND
Routing:
- net Net-(J2-Pin_9): track 7.34 -> 0.00 mm
- net GND: track 0.00 -> 7.34 mm
Other:
- board text added: "3.3V"
- board text added: "DIO0"
- board text added: "DIO1"
- board text added: "DIO10"
- board text added: "DIO11"
- board text added: "DIO3"
- board text added: "DIO5"
- board text added: "DIO6"
- board text added: "DIO7"
- board text added: "DIO8"
- board text added: "DIO9"
- board text added: "Designer: Rakshak Sudhakaran Date: 02/2025 Name: XBee Breakout Board RevA"
- board text added: "GND"
- board text added: "MISO"
- board text added: "MOSI"
- board text added: "RST"
- board text added: "Rx"
- board text added: "SCK"
- board text added: "Tx"
- board text added: "Vin"
- board text added: "Vout"
