File: hardware/XBeeBreakoutBoard/XBeeBreakoutBoard.kicad_sch (KiCad schematic)
At the start: 9 parts, among them J1 Conn_01x02, J2 Conn_01x10_Socket, J4 Conn_01x10_Socket, J5 Conn_01x05_Pin, U1 XB3-24Z8PT-J

Commit message: XBee Breakout production files
Connections:
- net GND: now also J2.9 (Pin_9), U1.10 (GND)
Changed lines of the file:
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@@
 (kicad_sch (version 20230121) (generator eeschema)
   (paper "A4")
+  (junction (at 204.47 99.06) (diameter 0) (color 0 0 0 0)
+  )
   (junction (at 170.18 62.23) (diameter 0) (color 0 0 0 0)
   )
@@
   (junction (at 204.47 38.1) (diameter 0) (color 0 0 0 0)
   )
-  (wire (pts (xy 196.85 96.52) (xy 207.01 96.52))
+  (wire (pts (xy 204.47 96.52) (xy 207.01 96.52))
     (stroke (width 0) (type default))
   )
@@
     (stroke (width 0) (type default))
   )
-  (wire (pts (xy 189.23 99.06) (xy 196.85 99.06))
+  (wire (pts (xy 189.23 99.06) (xy 204.47 99.06))
     (stroke (width 0) (type default))
   )
@@
     (stroke (width 0) (type default))
   )
-  (wire (pts (xy 196.85 99.06) (xy 196.85 96.52))
+  (wire (pts (xy 204.47 99.06) (xy 204.47 96.52))
     (stroke (width 0) (type default))
   )
@@
   )
   (symbol (lib_id "LD1117V33C:LD1117V33C") (at 181.61 59.69 0) (unit 1)
-    (in_bom yes) (on_board yes) (dnp no) (fields_autoplaced)
+    (in_bom yes) (on_board yes) (dnp no)
     (property "Reference" "CR1" (at 204.47 49.53 0)
       (effects (font (size 1.524 1.524)))
