File: hardware/DAQ_Module_CDR_Crunch/DAQ_module.kicad_sch (KiCad schematic)
At the start: 17 parts, among them J1 Conn_01x10_Pin, J2 Conn_01x10_Pin, J3 Conn_01x10_Pin, U1 MCP3564RT-E/ST, U2 MAX31855KASA, U3 MAX31855KASA, U7 TPS70933DBVR, U8 MAX31855KASA

Commit message: Ready for final review. Added downloadable footprint and symbol of board
Parts:
- removed J2, J3: Conn_01x10_Pin, Connector_PinHeader_2.54mm:PinHeader_1x10_P2.54mm_Vertical, symbol Connector:Conn_01x10_Pin
- added J3: Conn_01x20_Pin, Connector_PinHeader_2.54mm:PinHeader_1x20_P2.54mm_Vertical, symbol Connector:Conn_01x20_Pin
Connections:
- net +5V: now also J3.11 (Pin_11)
- net ADC_AI0: now also J3.1 (Pin_1)
- net ADC_AI1: now also J3.2 (Pin_2)
- net ADC_AI2: now also J3.3 (Pin_3)
- net ADC_AI3: now also J3.4 (Pin_4)
- net ADC_AI4: now also J3.5 (Pin_5)
- net ADC_AI5: now also J3.6 (Pin_6)
- net ADC_AI6: now also J3.7 (Pin_7)
- net ADC_AI7: now also J3.8 (Pin_8)
- net GND: now also C19.1, U7.2 (GND), J3.10 (Pin_10), J3.12 (Pin_12), J3.13 (Pin_13), J3.20 (Pin_20), J3.9 (Pin_9)
- net GPIO12 (CS_N20): now also J1.9 (Pin_9); no longer J1.8 (Pin_8)
- net GPIO13 (CS Chamber Shell_2): now also J1.8 (Pin_8); no longer J1.9 (Pin_9)
- net GPIO5 (CS_ADC): now also J1.4 (Pin_4); no longer J1.2 (Pin_2)
- net GPIO7 (MOSI_ADC): now also J1.2 (Pin_2); no longer J1.4 (Pin_4)
- net T+ (Chamber Shell_1): now also J3.15 (Pin_15)
- net T+ (Chamber Shell_2): now also J3.17 (Pin_17)
- net T+ (N2O): now also J3.19 (Pin_19)
- net T- (Chamber Shell_1): now also J3.14 (Pin_14)
- net T- (Chamber Shell_2): now also J3.16 (Pin_16)
- net T- (N2O): now also J3.18 (Pin_18)
Other:
- moved on the sheet: J1
